File: KiCad_Files/Wii_PCB/BROADWAY_GND.kicad_sch (KiCad schematic)
At the start: 1 part

Commit message: Updated RAM & GPU bus to allow custom net rules for measuring intra-track spacing, added pad for reset, removed debug pads, reorganized ram schematic to cluster length matched signals, changed MX chip and U10 symbols, and re-labeled the wifi net interface.
Parts:
- BROADWAY1: footprint wii_bgaLibrary:Updated BROADWAY -> WeeWii_Library:Updated BROADWAY
Changed lines of the file:
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@@
 			)
 		)
-		(property "Footprint" "wii_bgaLibrary:Updated BROADWAY"
+		(property "Footprint" "WeeWii_Library:Updated BROADWAY"
 			(at 140.97 6.35 0)
 			(effects
