File: KiCad_Files/Wii_PCB/HOLLYWOOD_GND.kicad_sch (KiCad schematic)
At the start: 1 part

Commit message: Updated RAM & GPU bus to allow custom net rules for measuring intra-track spacing, added pad for reset, removed debug pads, reorganized ram schematic to cluster length matched signals, changed MX chip and U10 symbols, and re-labeled the wifi net interface.
Parts:
- HOLLYWOOD1: footprint wii_bgaLibrary:Updated HOLLYWOOD -> WeeWii_Library:Updated HOLLYWOOD
Changed lines of the file:
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@@
 			)
 		)
-		(property "Footprint" "wii_bgaLibrary:Updated HOLLYWOOD"
+		(property "Footprint" "WeeWii_Library:Updated HOLLYWOOD"
 			(at 210.82 130.556 0)
 			(effects
@@
 		(pin "AE21"
 		)
-		(pin ""
+		(pin "N10"
 		)
 		(pin "A9"
@@
 		(pin "AG19"
 		)
-		(pin ""
+		(pin "B14"
 		)
 		(pin "AD16"
@@
 		(pin "C16"
 		)
-		(pin "D16"
+		(pin "E14"
 		)
 		(pin "W27"
@@
 		(pin "G11"
 		)
+		(pin "A24"
+		)
+		(pin "D19"
+		)
 		(instances
