File: KiCad_Files/Wii_PCB/HOLLYWOOD_IO.kicad_sch (KiCad schematic)
At the start: 28 parts, among them J1 Conn_01x20_Pin

Commit message: Updated RAM & GPU bus to allow custom net rules for measuring intra-track spacing, added pad for reset, removed debug pads, reorganized ram schematic to cluster length matched signals, changed MX chip and U10 symbols, and re-labeled the wifi net interface.
Parts:
- added J2: MSD-4-A, WeeWii_Library:MICROSD_MSD-4-A, symbol Wii_symbols:MICROSD-MSD-4-A
- added NT1: NetTie, NetTie:NetTie-2_SMD_Pad0.5mm, symbol Device:NetTie_2
- added R163: 10, Resistor_SMD:R_0402_1005Metric, symbol Device:R
- added R200: 47k, Resistor_SMD:R_0402_1005Metric, symbol Device:R
- added R21: 4.7k, Resistor_SMD:R_0402_1005Metric, symbol Device:R
- added R400, R401, R402, R403, R404, R405: 22, Resistor_SMD:R_0402_1005Metric, symbol Device:R
- added RESET1, TP0, TP1, TP2, TP3, TP4, TP5, TP6, TP7: TestPoint, TestPoint:TestPoint_Pad_D1.0mm, symbol Connector:TestPoint
- C63, C73, C89, C90, C94, C95, D3, D4, R51, U3: now left out of the parts list
- C70, C71, R36, R38, TPL1, TPR1: now fitted
- HOLLYWOOD1: footprint wii_bgaLibrary:Updated HOLLYWOOD -> WeeWii_Library:Updated HOLLYWOOD
- J1: footprint Connector_Molex:Molex_SlimStack_52991-0208_2x10_P0.50mm_Vertical -> WeeWii_Library:Molex_SlimStack_Wifi
Connections:
- net 3.3V: now also J1.11 (Pin_11), J1.12 (Pin_12), J2.4 (VDD), R200.2; no longer J1.18 (Pin_18), J1.20 (Pin_20)
- net BT: now also HOLLYWOOD1.B3 (BT_USB2); no longer HOLLYWOOD1.A3 (BT)
- net GND: now also J1.13 (Pin_13), J1.18 (Pin_18), J1.20 (Pin_20), J1.4 (Pin_4), J1.8 (Pin_8), J2.6 (VSS), J2.G1 (COVER_GND), J2.G2 (COVER_GND__1), J2.G3 (COVER_GND__2), J2.G4 (COVER_GND__3); no longer J1.11 (Pin_11), J1.12 (Pin_12), J1.16 (Pin_16), J1.2 (Pin_2), J1.7 (Pin_7)
- net SDA: now also R21.1
- net debug pad0: now also TP0.1
- net debug pad1: now also TP1.1
- net debug pad2: now also TP2.1
- net debug pad3: now also TP3.1
- net debug pad4: now also TP4.1
- net debug pad5: now also TP5.1
- net debug pad6: now also TP6.1
- net debug pad7: now also TP7.1
- net reset: now also RESET1.1
- net ~{BT}: now also HOLLYWOOD1.A3 (~{BT}_~{USB2}); no longer HOLLYWOOD1.B3 (~{BT})
- net R_WIFI_SDIO0: now reaches J1.17 (Pin_17)
- net R_WIFI_SDIO0: now also RA20_3.1
- net R_WIFI_SDIOCMD: now reaches J1.19 (Pin_19)
- net R_WIFI_SDIOCMD: now also RA20_2.1
- net DISC_DRIVE0 renamed DID7
- net DISC_DRIVE1 renamed DID6
- net DISC_DRIVE10 renamed DIBRK
- net DISC_DRIVE11 renamed DICOVER
- net DISC_DRIVE12 renamed ~{DIRST}
- net DISC_DRIVE13 renamed DID1
- net DISC_DRIVE14 renamed DID0
- net DISC_DRIVE15 renamed DIDIR
- net DISC_DRIVE16 renamed ~{DIHSTR}
- net DISC_DRIVE17 renamed ~{DIDSTR}
- net DISC_DRIVE18 renamed NOSPINUP
- net DISC_DRIVE2 renamed AISCLK
- net DISC_DRIVE3 renamed AISD
- net DISC_DRIVE4 renamed DID5
- net DISC_DRIVE5 renamed DID4
- net DISC_DRIVE6 renamed AISLR
- net DISC_DRIVE7 renamed ~{DIERR}
- net DISC_DRIVE8 renamed DID3
- net DISC_DRIVE9 renamed DID2
- net GC_CARD_P1 renamed A_SEN
- net GC_CARD_P11 renamed A_CLK
- net GC_CARD_P13 renamed B_SEN
- net GC_CARD_P15 renamed B_INT
- net GC_CARD_P17 renamed B_DIN
- net GC_CARD_P19 renamed B_DOUT
- net GC_CARD_P21 renamed B_CS
- net GC_CARD_P23 renamed B_CLK
- net GC_CARD_P3 renamed A_INT
- net GC_CARD_P5 renamed A_DIN
- net GC_CARD_P7 renamed A_DOUT
- net GC_CARD_P9 renamed A_CS
- net PIN16 renamed WIFI_SDIO3
- net PIN17 renamed WIFI_SDIO0
- net PIN19 renamed WIFI_SDIOCMD
- net PIN2 renamed WIFI_SDIO2
- net PIN3 renamed WIFI_SDIO1
- net PIN5 renamed WIFI_SDIOCLK
- net W_R16: no longer names the net of J1.10 (Pin_10)
- net W_R16: no longer RA20_4.1
- removed net W_R17: J1.8 (Pin_8), RA20_3.1
- removed net W_R19: J1.4 (Pin_4), RA20_2.1
- net W_R2 renamed R_WIFI_SDIO1
- net R_WIFI_SDIO1: now also R213.1; no longer R212.1
- net W_R3 renamed R_WIFI_SDIOCLK
- net R_WIFI_SDIOCLK: now also RA20_1.1; no longer R213.1
- net W_R5: no longer names the net of J1.9 (Pin_9)
- net W_R5: no longer RA20_1.1
- net mx_pin11 renamed GPU_EXI0_DO
- net mx_pin12 renamed GPU_EXI0_DI
- net mx_pin13 renamed GPU_EXI0_~{CS}
- net mx_pin14 renamed GPU_EXI0_CLK
- net mx_pin24 renamed Delay_Enable
- net sd_data1 renamed SD_CMD
- net SD_CMD: now also R404.2
- net sd_data2 renamed SD_DAT3
- net SD_DAT3: now also R403.2
- net sd_data3 renamed SD_DAT2
- net SD_DAT2: now also R402.2
- net sd_data4 renamed SD_CLK
- net SD_CLK: now also R163.2
- net sd_data5 renamed SD_WP
- net SD_WP: now also NT1.2, R405.2
- net sd_data6 renamed SD_CD
- net SD_CD: now also NT1.1
- net sd_data7 renamed SD_DAT1
- net SD_DAT1: now also R401.2
- net sd_data8 renamed SD_DAT0
- net SD_DAT0: now also R400.2
- new net 1.8V: R21.2
- new net R_CARD_SENSE: J2.CD, R200.1, R405.1
- new net R_SD_CLK: J2.5 (CLK), R163.1
- new net R_SD_CMD: J2.3 (CMD), R404.1
- new net R_SD_DAT0: J2.7 (DAT0), R400.1
- new net R_SD_DAT1: J2.8 (DAT1), R401.1
- new net R_SD_DAT2: J2.1 (DAT2), R402.1
- new net R_SD_DAT3: J2.2 (CD/DAT3), R403.1
- new net R_WIFI_SDIO2: J1.2 (Pin_2), R212.1
- new net R_WIFI_SDIO3: J1.16 (Pin_16), RA20_4.1
- no-connect marks 82 -> 83
Other:
- note added: "MICRO SD Card"
- note added: "R200/R201 consolidated to one pullup"
- note added: "Regular signals (RA10/RA11) Renamed to R400-R404 WP_CD Merged into R405 16.7R -> 22R SD_CLK remains 10R, same name"
- note added: "TEST POINTS"
- moved on the sheet: HOLLYWOOD1G, R212, R213, RA20_1, RA20_2, RA20_3, RA20_4
