File: KiCad_Files/Wii_PCB/HOLLYWOOD_VCC.kicad_sch (KiCad schematic)
At the start: 1 part

Commit message: Updated RAM & GPU bus to allow custom net rules for measuring intra-track spacing, added pad for reset, removed debug pads, reorganized ram schematic to cluster length matched signals, changed MX chip and U10 symbols, and re-labeled the wifi net interface.
Parts:
- HOLLYWOOD1: footprint wii_bgaLibrary:Updated HOLLYWOOD -> WeeWii_Library:Updated HOLLYWOOD
Changed lines of the file:
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@@
 			)
 		)
-		(property "Footprint" "wii_bgaLibrary:Updated HOLLYWOOD"
+		(property "Footprint" "WeeWii_Library:Updated HOLLYWOOD"
 			(at 288.29 112.776 0)
 			(effects
@@
 		(pin "A6"
 		)
-		(pin ""
-		)
-		(pin ""
-		)
 		(pin "B6"
 		)
@@
 		(pin "F27"
 		)
-		(pin "D16"
-		)
 		(pin "A11"
